File: Rx_Preamp/Rx_Preamp.sch (KiCad schematic (older format))
At the start: 74 parts, among them J1 Conn_Coaxial, J2 Conn_Coaxial, SW1 SW_DIP_x04, U1 AD8429, U2 LT6350HMS8TRPBF, U7 ADA4610-1ARJZ, U8 PIG-LOGO, U9 PIG-LOGO

Commit message: Update Preamp files
Parts:
- removed C?: 62p, Capacitor_SMD:C_1206_3216Metric, symbol Device:C
- removed D? (x3): BAV99, Package_TO_SOT_SMD:SOT-23, symbol Diode:BAV99
- added C5, C6: 300p, Capacitor_SMD:C_1206_3216Metric, symbol Device:C
- added D7, D8: D, Diode_SMD:D_SMB, symbol Device:D
- added R10, R14, R15, R9: 1k, Resistor_SMD:R_1206_3216Metric, symbol Device:R
- added TP10, TP11: TestPoint, TestPoint:TestPoint_THTPad_1.0x1.0mm_Drill0.5mm, symbol Connector:TestPoint
- added U3, U4: ADA4610-1ARJZ, Package_TO_SOT_SMD:SOT-23-5, symbol Rx_Preamp-rescue:ADA4610-1ARJZ-LT1010
- R16, R17: value 47 -> 49.9
Connections:
- net +5V: now also U3.5 (V+), U4.5 (V+)
- net -5V: now also U3.2 (V-), U4.2 (V-)
- net GND: now also U3.3 (+), U4.3 (+)
- net SE2D-Out1: now also R9.1; no longer R16.1
- net SE2D-Out2: now also R10.1; no longer R17.1
- net SigFilt+: now also D7.1 (K), D8.2 (A)
- net SigFilt-: now also D7.2 (A), D8.1 (K)
- new net Out1-AmpOut: C5.1, R14.2, R16.1, TP10.1, U3.1
- new net Out1-AmpV-: C5.2, R14.1, R9.2, U3.4 (-)
- new net Out2-AmpOut: C6.1, R15.2, R17.1, TP11.1, U4.1
- new net Out2-AmpV-: C6.2, R10.2, R15.1, U4.4 (-)
Other:
- moved on the sheet: J1, J2, R16, R17
